File: Moco-IOBreakoutPCB.kicad_sch (KiCad schematic)
At the start: 6 parts, among them J1 Conn_01x14, J2 Conn_01x14, J3 Conn_01x06, J4 Conn_01x06, J5 Conn_01x06, J6 Conn_01x06

Commit message: layout
Parts:
- removed J6: Conn_01x06, symbol Connector_Generic:Conn_01x06
- J1, J2: footprint (none) -> UTSVT_Connectors:Molex_Microfit3.0_02x07_14-Pin-Vertical-PCB-Receptacle_447691401
- J3, J4, J5: footprint (none) -> UTSVT_Connectors:Molex_Microfit3.0_02x03_6-Pin-Vertical-PCB-Receptacle_447690601
Connections:
- net Serial_RX+: now reaches J1.1 (Pin_1)
- net Serial_RX+: now also J2.1 (Pin_1)
- net H2/B_RX-: now reaches J1.10 (Pin_10)
- net H2/B_RX-: now also J2.10 (Pin_10)
- net H1/A_RX-: now reaches J1.11 (Pin_11)
- net H1/A_RX-: now also J2.11 (Pin_11)
- net GND_MCI: now reaches J1.12 (Pin_12)
- net GND_MCI: now also J1.13 (Pin_13), J2.12 (Pin_12), J2.13 (Pin_13)
- net Shield_MCI: now reaches J1.14 (Pin_14)
- net Shield_MCI: now also J2.14 (Pin_14)
- net H3/I_RX+: now reaches J1.2 (Pin_2)
- net H3/I_RX+: now also J2.2 (Pin_2)
- net H2/B_RX+: now reaches J1.3 (Pin_3)
- net H2/B_RX+: now also J2.3 (Pin_3)
- net H1/A_RX+: now reaches J1.4 (Pin_4)
- net H1/A_RX+: now also J2.4 (Pin_4)
- net +12V_MCI: now reaches J1.5 (Pin_5)
- net +12V_MCI: now also J2.5 (Pin_5)
- net +5V_MCI: now reaches J1.6 (Pin_6)
- net +5V_MCI: now also J2.6 (Pin_6)
- net Serial_RX-: now reaches J1.8 (Pin_8)
- net Serial_RX-: now also J2.8 (Pin_8)
- net H3/I_RX-: now reaches J1.9 (Pin_9)
- net H3/I_RX-: now also J2.9 (Pin_9)
- net +12V: now reaches J5.1 (Pin_1)
- net +12V: now also J3.1 (Pin_1)
- net GND: now reaches J5.2 (Pin_2)
- net GND: now also J3.2 (Pin_2)
- net CAN_H-in: now reaches J5.3 (Pin_3)
- net CAN_H-in: now also J3.4 (Pin_4)
- net CAN_L-in: now reaches J5.4 (Pin_4)
- net CAN_L-in: now also J3.5 (Pin_5)
- net CAN_H-out: now reaches J5.5 (Pin_5)
- net CAN_H-out: now also J4.4 (Pin_4)
- net CAN_L-out: now reaches J5.6 (Pin_6)
- net CAN_L-out: now also J4.5 (Pin_5)
- no-connect marks 0 -> 8
Other:
- moved on the sheet: J2, J3, J4, J5

Commit message: 120 ohm terminating microphone condenser
Parts:
- added 120m/s1: Microphone_Condenser, Resistor_SMD:R_0603_1608Metric, symbol Device:Microphone_Condenser
Connections:
- net CAN_H-out: now also 120m/s1.1 (-)
- net CAN_L-out: now also 120m/s1.2 (+)
Changed lines of the file:
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@@
+	(wire
+		(pts
+			(xy 138.43 121.92) (xy 138.43 128.27)
+		)
+		(stroke
+			(width 0)
+			(type default)
+		)
+	)
 	(wire
 		(pts
@@
 		(pts
 			(xy 82.55 100.33) (xy 93.98 100.33)
+		)
+		(stroke
+			(width 0)
+			(type default)
+		)
+	)
+	(wire
+		(pts
+			(xy 138.43 107.95) (xy 138.43 111.76)
 		)
 		(stroke
@@
 		)
 	)
+	(label "CAN_H-out"
+		(at 138.43 128.27 180)
+		(effects
+			(font
+				(size 1.27 1.27)
+			)
+			(justify right bottom)
+		)
+	)
 	(label "H3{slash}I_RX+"
 		(at 50.8 39.37 180)
+		(effects
+			(font
+				(size 1.27 1.27)
+			)
+			(justify right bottom)
+		)
+	)
+	(label "CAN_L-out"
+		(at 138.43 107.95 180)
 		(effects
 			(font
@@
 					(unit 1)
 				)
+			)
+		)
+	)
+	(symbol
+		(lib_id "Device:Microphone_Condenser")
+		(at 138.43 116.84 0)
+		(unit 1)
+		(exclude_from_sim no)
+		(in_bom yes)
+		(on_board yes)
+		(dnp no)
+		(fields_autoplaced yes)
+		(property "Reference" "120m/s1"
+			(at 142.24 114.8714 0)
+			(effects
+				(font
+					(size 1.27 1.27)
+				)
+				(justify left)
+			)
+		)
+		(property "Value" "Microphone_Condenser"
+			(at 142.24 117.4114 0)
+			(effects
+				(font
+					(size 1.27 1.27)
+				)
+				(justify left)
+			)
+		)
+		(property "Footprint" "Resistor_SMD:R_0603_1608Metric"
+			(at 138.43 114.3 90)
+			(effects
+				(font
+					(size 1.27 1.27)
+				)
+				(hide yes)
+			)
+		)
+		(property "Datasheet" "~"
+			(at 138.43 114.3 90)
+			(effects
+				(font
+					(size 1.27 1.27)
+				)
+				(hide yes)
+			)
+		)
+		(property "Description" "Condenser microphone"
+			(at 138.43 116.84 0)
+			(effects
+				(font
+					(size 1.27 1.27)
+				)
+				(hide yes)
+			)
+		)
+		(pin "2"
+		)
+		(pin "1"
+		)
+		(instances
+			(project ""
+				(path "/4d2355e5-c5e4-41a8-8c49-cd06df0eb21b"
+					(reference "120m/s1")
+					(unit 1)
+				)
