File: Moco-IOBreakoutPCB.kicad_pcb (KiCad board)
At the start: 2 copper layers, 67.5 x 45.5 mm, 7 parts, among them J1 Conn_01x14, J2 Conn_01x14, J3 Conn_01x06, J4 Conn_01x06, J5 Conn_01x06

Commit message: routing
Routing:
- net /Serial_RX+: track 0.00 -> 47.0 mm
- net /CAN_H-in: track 0.00 -> 46.7 mm
- net /Serial_RX-: track 0.00 -> 45.3 mm
- net /H3/I_RX+: track 0.00 -> 42.8 mm
- net GND_MCI: track 0.00 -> 42.2 mm
- net +12V: track 0.00 -> 41.6 mm
- net /H3/I_RX-: track 0.00 -> 41.5 mm
- net /H2/B_RX+: track 0.00 -> 38.5 mm
- net /H2/B_RX-: track 0.00 -> 37.5 mm
- net +5V_MCI: track 0.00 -> 37.2 mm
- net /CAN_L-in: track 0.00 -> 36.8 mm
- net /H1/A_RX+: track 0.00 -> 36.5 mm
- net /Shield_MCI: track 0.00 -> 36.2 mm
- net /H1/A_RX-: track 0.00 -> 35.6 mm
- net +12V_MCI: track 0.00 -> 35.3 mm
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- added copper zone on B.Cu, net GND
- added copper zone on F.Cu, net GND

Commit message: 120 ohm terminating microphone condenser
Parts:
- added 120m/s1: Microphone_Condenser, Resistor_SMD:R_0603_1608Metric, F.Cu at (142.9, 66.2)
Routing:
- net /CAN_H-out: track 26.8 -> 36.3 mm
- net /CAN_L-out: track 25.8 -> 34.7 mm

Commit message: type shi
Parts:
- moved 120m/s1 0.55 mm to (142.9, 66.8)
Routing:
- net +12V: track 41.6 -> 41.0 mm
- net /CAN_L-out: track 34.7 -> 34.2 mm
